File: hardware/Charge Controller Files (Michael, Sky)/ChargeController2.0.kicad_sch (KiCad schematic)
At the start: 72 parts, among them J10 Conn-1x2, J11 Conn-1x2, J12 Conn-1x2, J13 Conn-1x2, J14 Conn-1x2, J15 Conn-1x2, J16 Conn-1x2, J2 Conn_01x02_Pin, J3 Conn-1x2, J6 Conn-1x2, J7 Conn-1x2, J8 Conn-1x2, J9 Conn-1x2, Q5 AONS66614, Q6 AONS66614, Q7 AONS66614, Q8 AONS66614, U1 BQ25756RRVR

Commit message: added symbol files
Parts:
- added R11: 10, symbol Device:R
Connections:
- net DRV_SUP: now also R11.1
- net REGN: now also R11.2
- net Next renamed Main
Other:
- note added: "Bi-Directional Buck-Boost Converter"
- note added: "MAIN"
- note removed: "Buck Boost Converter"
- moved on the sheet: C3
Changed lines of the file:
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@@
 		)
 	)
-	(text "Buck Boost Converter"
+	(text "MAIN"
 		(exclude_from_sim no)
-		(at 87.376 13.97 0)
+		(at 240.792 95.758 0)
+		(effects
+			(font
+				(size 1.27 1.27)
+			)
+		)
+	)
+	(text "Bi-Directional Buck-Boost Converter"
+		(exclude_from_sim no)
+		(at 94.234 14.224 0)
 		(effects
 			(font
@@
 	)
 	(junction
+		(at 191.77 113.03)
+		(diameter 0)
+		(color 0 0 0 0)
+	)
+	(junction
 		(at 210.82 138.43)
 		(diameter 0)
@@
 	)
 	(junction
-		(at 189.23 138.43)
+		(at 191.77 120.65)
 		(diameter 0)
 		(color 0 0 0 0)
 	)
 	(junction
-		(at 193.04 115.57)
+		(at 189.23 138.43)
 		(diameter 0)
 		(color 0 0 0 0)
@@
 	(wire
 		(pts
+			(xy 186.69 120.65) (xy 191.77 120.65)
+		)
+		(stroke
+			(width 0)
+			(type default)
+		)
+	)
+	(wire
+		(pts
 			(xy 53.34 162.56) (xy 53.34 158.75)
 		)
@@
 	(wire
 		(pts
-			(xy 193.04 127) (xy 193.04 128.27)
+			(xy 191.77 129.54) (xy 191.77 130.81)
 		)
 		(stroke
@@
 	(wire
 		(pts
+			(xy 213.36 115.57) (xy 198.12 115.57)
+		)
+		(stroke
+			(width 0)
+			(type default)
+		)
+	)
+	(wire
+		(pts
 			(xy 273.05 143.51) (xy 269.24 143.51)
 		)
@@
 	(wire
 		(pts
+			(xy 198.12 120.65) (xy 191.77 120.65)
+		)
+		(stroke
+			(width 0)
+			(type default)
+		)
+	)
+	(wire
+		(pts
 			(xy 177.8 81.28) (xy 177.8 83.82)
 		)
@@
 	(wire
 		(pts
-			(xy 193.04 115.57) (xy 193.04 119.38)
-		)
-		(stroke
-			(width 0)
-			(type default)
-		)
-	)
-	(wire
-		(pts
 			(xy 132.08 125.73) (xy 130.81 125.73)
 		)
@@
 	(wire
 		(pts
+			(xy 191.77 113.03) (xy 213.36 113.03)
+		)
+		(stroke
+			(width 0)
+			(type default)
+		)
+	)
+	(wire
+		(pts
 			(xy 27.94 17.78) (xy 24.13 17.78)
 		)
@@
 	(wire
 		(pts
-			(xy 146.05 55.88) (xy 146.05 54.61)
+			(xy 198.12 115.57) (xy 198.12 120.65)
 		)
 		(stroke
@@
 	(wire
 		(pts
-			(xy 41.91 76.2) (xy 45.72 76.2)
+			(xy 146.05 55.88) (xy 146.05 54.61)
 		)
 		(stroke
@@
 	(wire
 		(pts
-			(xy 29.21 107.95) (xy 29.21 130.81)
+			(xy 41.91 76.2) (xy 45.72 76.2)
 		)
 		(stroke
@@
 	(wire
 		(pts
-			(xy 175.26 48.26) (xy 179.07 48.26)
+			(xy 29.21 107.95) (xy 29.21 130.81)
 		)
 		(stroke
@@
 	(wire
 		(pts
-			(xy 242.57 46.99) (xy 254 46.99)
+			(xy 175.26 48.26) (xy 179.07 48.26)
 		)
 		(stroke
@@
 	(wire
 		(pts
-			(xy 190.5 111.76) (xy 190.5 113.03)
+			(xy 242.57 46.99) (xy 254 46.99)
 		)
 		(stroke
@@
 	(wire
 		(pts
-			(xy 189.23 115.57) (xy 193.04 115.57)
+			(xy 190.5 111.76) (xy 190.5 113.03)
 		)
 		(stroke
@@
 	(wire
 		(pts
-			(xy 190.5 113.03) (xy 213.36 113.03)
+			(xy 190.5 113.03) (xy 191.77 113.03)
 		)
 		(stroke
@@
 	(wire
 		(pts
-			(xy 193.04 115.57) (xy 213.36 115.57)
-		)
-		(stroke
-			(width 0)
-			(type default)
-		)
-	)
-	(wire
-		(pts
 			(xy 95.25 186.69) (xy 95.25 180.34)
 		)
@@
 	(wire
 		(pts
+			(xy 191.77 120.65) (xy 191.77 121.92)
+		)
+		(stroke
+			(width 0)
+			(type default)
+		)
+	)
+	(wire
+		(pts
 			(xy 105.41 43.18) (xy 105.41 46.99)
 		)
@@
 		)
 	)
-	(label "Next"
+	(label "Main"
 		(at 167.64 116.84 0)
 		(effects
@@
 		)
 	)
-	(label "Next"
+	(label "Main"
 		(at 82.55 27.94 180)
 		(effects
@@
 	)
 	(label "REGN"
-		(at 189.23 115.57 180)
+		(at 186.69 120.65 180)
 		(effects
 			(font
@@
 	(symbol
 		(lib_id "power:GND")
-		(at 193.04 128.27 0)
+		(at 191.77 130.81 0)
 		(unit 1)
 		(exclude_from_sim no)
@@
 		(fields_autoplaced yes)
 		(property "Reference" "#PWR07"
-			(at 193.04 134.62 0)
+			(at 191.77 137.16 0)
 			(effects
 				(font
@@
 		)
 		(property "Value" "GND"
-			(at 193.04 133.35 0)
+			(at 191.77 135.89 0)
 			(effects
 				(font
@@
 		)
 		(property "Footprint" ""
-			(at 193.04 128.27 0)
+			(at 191.77 130.81 0)
 			(effects
 				(font
@@
 		)
 		(property "Datasheet" ""
-			(at 193.04 128.27 0)
+			(at 191.77 130.81 0)
 			(effects
 				(font
@@
 		)
 		(property "Description" "Power symbol creates a global label with name \"GND\" , ground"
-			(at 193.04 128.27 0)
+			(at 191.77 130.81 0)
 			(effects
 				(font
@@
 	(symbol
 		(lib_id "Device:C")
-		(at 193.04 123.19 0)
+		(at 191.77 125.73 0)
 		(unit 1)
 		(exclude_from_sim no)
@@
 		(dnp no)
 		(property "Reference" "C3"
-			(at 187.706 121.412 0)
+			(at 186.436 123.952 0)
 			(effects
 				(font
@@
 		)
 		(property "Value" "4.7u"
-			(at 186.436 123.698 0)
+			(at 185.166 126.238 0)
 			(effects
 				(font
@@
 		)
 		(property "Footprint" ""
-			(at 194.0052 127 0)
+			(at 192.7352 129.54 0)
 			(effects
 				(font
@@
 		)
 		(property "Datasheet" "~"
-			(at 193.04 123.19 0)
+			(at 191.77 125.73 0)
 			(effects
 				(font
@@
 		)
 		(property "Description" "Unpolarized capacitor"
-			(at 193.04 123.19 0)
+			(at 191.77 125.73 0)
 			(effects
 				(font
@@
 					(unit 1)
 				)
+			)
+		)
+	)
+	(symbol
+		(lib_id "Device:R")
+		(at 191.77 116.84 0)
+		(unit 1)
+		(exclude_from_sim no)
+		(in_bom yes)
+		(on_board yes)
+		(dnp no)
+		(property "Reference" "R11"
+			(at 193.04 115.316 0)
+			(effects
+				(font
+					(size 1.27 1.27)
+				)
+				(justify left)
+			)
+		)
+		(property "Value" "10"
+			(at 193.548 118.11 0)
+			(effects
+				(font
+					(size 1.27 1.27)
+				)
+				(justify left)
+			)
+		)
+		(property "Footprint" ""
+			(at 189.992 116.84 90)
+			(effects
+				(font
+					(size 1.27 1.27)
+				)
+				(hide yes)
+			)
+		)
+		(property "Datasheet" "~"
+			(at 191.77 116.84 0)
+			(effects
+				(font
+					(size 1.27 1.27)
+				)
+				(hide yes)
+			)
+		)
+		(property "Description" "Resistor"
+			(at 191.77 116.84 0)
+			(effects
+				(font
+					(size 1.27 1.27)
+				)
+				(hide yes)
+			)
+		)
+		(pin "1"
+		)
+		(pin "2"
+		)
+		(instances
+			(project ""
+				(path "/89a953c5-1b9f-4ec7-83f7-649f6dcfa61f"
+					(reference "R11")
+					(unit 1)
+				)
