File: hardware/Charge Controller Files (Parsa)/Charge Controller.kicad_sch (KiCad schematic)
At the start: 55 parts, among them J1 61300311121, J2 Conn_01x02_Pin, Q1 AONS66614, Q2 AONS66614, Q3 AONS66614, Q4 AONS66614, U1 BQ25756RRVR

Commit message: added symbol files
Changed lines of the file:
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@@
 (kicad_sch
-	(version 20231120)
+	(version 20250114)
 	(generator "eeschema")
-	(generator_version "8.0")
+	(generator_version "9.0")
 	(paper "A3")
 	(junction
@@
 		)
 	)
+	(embedded_fonts no)
 )
