File: hardware/Charge Controller Files (Michael)/_autosave-ChargeController2.0.kicad_sch (KiCad schematic)
At the start: 82 parts, among them J1 Conn_01x02_Pin, J10 Conn-1x2, J11 Conn-1x2, J12 Conn-1x2, J13 Conn-1x2, J14 Conn-1x2, J15 Conn-1x2, J16 Conn-1x2, J17 SCL_MAS_01x01_Pin, J18 SDA_MAS_01x01_Pin, J2 SP_01x02_Pin, J3 SYS-1x2, J4 3.3V_PULLUP_01x01_Pin, J5 BATT_01x02_Pin, J6 Conn-1x2, J7 Conn-1x2, J8 Conn-1x2, J9 Conn-1x2, Q5 AONS66614, Q6 AONS66614, Q7 AONS66614, Q8 AONS66614, U1 BQ25756RRVR

Commit message: More design
Design Specs IV
Parts:
- removed J1: Conn_01x02_Pin, symbol Connector:Conn_01x02_Pin
Changed lines of the file:
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@@
 	)
 	(junction
-		(at 106.68 190.5)
-		(diameter 0)
-		(color 0 0 0 0)
-	)
-	(junction
 		(at 74.93 60.96)
 		(diameter 0)
@@
 	)
 	(junction
-		(at 106.68 167.64)
-		(diameter 0)
-		(color 0 0 0 0)
-	)
-	(junction
 		(at 259.08 35.56)
 		(diameter 0)
@@
 	(wire
 		(pts
-			(xy 118.11 167.64) (xy 106.68 167.64)
-		)
-		(stroke
-			(width 0)
-			(type default)
-		)
-	)
-	(wire
-		(pts
 			(xy 198.12 137.16) (xy 184.15 137.16)
 		)
@@
 	(wire
 		(pts
-			(xy 106.68 190.5) (xy 118.11 190.5)
-		)
-		(stroke
-			(width 0)
-			(type default)
-		)
-	)
-	(wire
-		(pts
 			(xy 163.83 73.66) (xy 163.83 77.47)
 		)
@@
 	(wire
 		(pts
-			(xy 118.11 186.69) (xy 118.11 190.5)
-		)
-		(stroke
-			(width 0)
-			(type default)
-		)
-	)
-	(wire
-		(pts
 			(xy 223.52 91.44) (xy 223.52 101.6)
 		)
@@
 	(wire
 		(pts
-			(xy 118.11 184.15) (xy 118.11 167.64)
-		)
-		(stroke
-			(width 0)
-			(type default)
-		)
-	)
-	(wire
-		(pts
 			(xy 265.43 163.83) (xy 266.7 163.83)
 		)
@@
 					(unit 1)
 				)
-			)
-		)
-	)
-	(symbol
-		(lib_id "Connector:Conn_01x02_Pin")
-		(at 113.03 184.15 0)
-		(unit 1)
-		(exclude_from_sim no)
-		(in_bom yes)
-		(on_board yes)
-		(dnp no)
-		(property "Reference" "J1"
-			(at 122.174 183.134 0)
-			(effects
-				(font
-					(size 1.27 1.27)
-				)
-			)
-		)
-		(property "Value" "Conn_01x02_Pin"
-			(at 127 186.69 0)
-			(effects
-				(font
-					(size 1.27 1.27)
-				)
-			)
-		)
-		(property "Footprint" ""
-			(at 113.03 184.15 0)
-			(effects
-				(font
-					(size 1.27 1.27)
-				)
-				(hide yes)
-			)
-		)
-		(property "Datasheet" "~"
-			(at 113.03 184.15 0)
-			(effects
-				(font
-					(size 1.27 1.27)
-				)
-				(hide yes)
-			)
-		)
-		(property "Description" "Generic connector, single row, 01x02, script generated"
-			(at 113.03 184.15 0)
-			(effects
-				(font
-					(size 1.27 1.27)
-				)
-				(hide yes)
-			)
-		)
-		(pin "2"
-		)
-		(pin "1"
-		)
-		(instances
-			(project ""
-				(path "/89a953c5-1b9f-4ec7-83f7-649f6dcfa61f"
-					(reference "J1")
-					(unit 1)
-				)
