File: hardware/Charge Controller Files (Michael)/ChargeController2.0.kicad_pcb (KiCad board)
At the start: 2 copper layers, 0 parts

Commit message: updated footprints
Parts:
- added C12: 56u, Capacitor_SMD:C_0201_0603Metric, F.Cu at (166.5, 88.5)
- added C13: 56u, Capacitor_SMD:C_0201_0603Metric, F.Cu at (166.5, 90.2)
- added C14: 100n, Capacitor_SMD:C_0402_1005Metric, F.Cu at (123.7, 98.9)
- added C15: 470n, Capacitor_SMD:C_0402_1005Metric, F.Cu at (123.7, 100.9)
- added C16: 100n, Capacitor_SMD:C_0402_1005Metric, F.Cu at (126.6, 97.0)
- added C17: 56u, Capacitor_SMD:C_0201_0603Metric, F.Cu at (166.5, 92.0)
- added C18: 56u, Capacitor_SMD:C_0201_0603Metric, F.Cu at (166.5, 93.7)
- added C19: 100n, Capacitor_SMD:C_0402_1005Metric, F.Cu at (126.6, 98.9)
- added C2: 56u, Capacitor_SMD:C_0201_0603Metric, F.Cu at (166.5, 86.7)
- added C20: 100n, Capacitor_SMD:C_0402_1005Metric, F.Cu at (126.6, 100.9)
- added C22: 4.7u, Capacitor_SMD:C_0603_1608Metric, F.Cu at (158.1, 77.1)
- added C23: 1u, Capacitor_SMD:C_0201_0603Metric, F.Cu at (166.5, 95.5)
- added C24: 56u, Capacitor_SMD:C_0201_0603Metric, F.Cu at (166.5, 97.2)
- added C25: 100n, Capacitor_SMD:C_0402_1005Metric, F.Cu at (129.5, 97.0)
- added C26: 470n, Capacitor_SMD:C_0402_1005Metric, F.Cu at (129.5, 98.9)
- added C27: 100n, Capacitor_SMD:C_0402_1005Metric, F.Cu at (129.5, 100.9)
- added C3: 4.7u, Capacitor_SMD:C_0603_1608Metric, F.Cu at (158.1, 69.5)
- added C4: 100n, Capacitor_SMD:C_0402_1005Metric, F.Cu at (123.7, 97.0)
- added C6: 47u, Capacitor_SMD:C_0603_1608Metric, F.Cu at (158.1, 72.0)
- added C7: 4.7u, Capacitor_SMD:C_0603_1608Metric, F.Cu at (158.1, 74.5)
- added D1: GREEN, LED_SMD:LED_0603_1608Metric, F.Cu at (132.9, 97.3)
- added D2: GREEN, LED_SMD:LED_0603_1608Metric, F.Cu at (132.9, 99.8)
- added D3: GREEN, LED_SMD:LED_0603_1608Metric, F.Cu at (132.9, 102.4)
- added D4: D, bmsfootprints:DO-214AC, F.Cu at (152.7, 70.2)
- added D5: D, bmsfootprints:DO-214AC, F.Cu at (152.7, 74.2)
- added D6: D, bmsfootprints:DO-214AC, F.Cu at (152.7, 78.1)
- added D7: D, bmsfootprints:DO-214AC, F.Cu at (152.7, 82.1)
- added D8: D, bmsfootprints:DO-214AC, F.Cu at (152.7, 86.0)
- added D9: D, bmsfootprints:DO-214AC, F.Cu at (152.7, 89.9)
- added H1: MountingHole_Pad, MountingHole:MountingHole_3.2mm_M3_ISO14580_Pad, F.Cu at (145.5, 71.8)
- added H2: MountingHole_Pad, MountingHole:MountingHole_3.2mm_M3_ISO14580_Pad, F.Cu at (145.5, 78.8)
- added H3: MountingHole_Pad, MountingHole:MountingHole_3.2mm_M3_ISO14580_Pad, F.Cu at (145.5, 85.9)
- added H4: MountingHole_Pad, MountingHole:MountingHole_3.2mm_M3_ISO14580_Pad, F.Cu at (145.5, 93.0)
- added J1: GND_TEST_01x01_Pin, Connector_PinHeader_2.54mm:PinHeader_1x01_P2.54mm_Vertical, F.Cu at (158.3, 88.1)
- added J10: SOL_TEST_01x01_Pin, Connector_PinHeader_2.54mm:PinHeader_1x01_P2.54mm_Vertical, F.Cu at (162.9, 88.1)
- added J13: Conn-1x2, Connector_PinHeader_2.54mm:PinHeader_1x02_P2.54mm_Vertical, F.Cu at (147.5, 54.2)
- added J14: Conn-1x2, Connector_PinHeader_2.54mm:PinHeader_1x02_P2.54mm_Vertical, F.Cu at (152.1, 54.2)
- added J15: Conn-1x2, Connector_PinHeader_2.54mm:PinHeader_1x02_P2.54mm_Vertical, F.Cu at (156.7, 54.2)
- added J17: SCL_MAS_01x01_Pin, Connector_PinHeader_2.54mm:PinHeader_1x01_P2.54mm_Vertical, F.Cu at (162.9, 92.7)
- added J18: SDA_MAS_01x01_Pin, Connector_PinHeader_2.54mm:PinHeader_1x01_P2.54mm_Vertical, F.Cu at (162.9, 97.3)
- added J19: SYS-1x2, Connector_PinHeader_2.54mm:PinHeader_1x02_P2.54mm_Vertical, F.Cu at (161.3, 54.2)
- added J2: SP_01x02_Pin, Connector_PinHeader_2.54mm:PinHeader_1x02_P2.54mm_Vertical, F.Cu at (124.6, 54.2)
- added J3: BATT_TEST_01x01_Pin, Connector_PinHeader_2.54mm:PinHeader_1x01_P2.54mm_Vertical, F.Cu at (158.3, 92.7)
- added J4: 3.3V_PULLUP_01x02_Pin, Connector_PinHeader_2.54mm:PinHeader_1x02_P2.54mm_Vertical, F.Cu at (129.2, 54.2)
- added J5: BATT_01x02_Pin, Connector_PinHeader_2.54mm:PinHeader_1x01_P2.54mm_Vertical, F.Cu at (158.3, 97.3)
- added J6: Conn-1x2, Connector_PinHeader_2.54mm:PinHeader_1x02_P2.54mm_Vertical, F.Cu at (133.8, 54.2)
- added J7: Conn-1x2, Connector_PinHeader_2.54mm:PinHeader_1x02_P2.54mm_Vertical, F.Cu at (138.4, 54.2)
- added J8: Conn-1x2, Connector_PinHeader_2.54mm:PinHeader_1x02_P2.54mm_Vertical, F.Cu at (142.9, 54.2)
- added J9: SYS_TEST_01x01_Pin, Connector_PinHeader_2.54mm:PinHeader_1x01_P2.54mm_Vertical, F.Cu at (158.3, 101.9)
- added L1: IHLP6767GZER100M01, bmsfootprints:IND_IHLP6767GZER100M01, F.Cu at (132.2, 77.6)
- added Q1: SI2318DS-T1-E3, bmsfootprints:SI2318DS-T1-E3, F.Cu at (158.0, 61.3)
- added Q10: SI2318DS-T1-E3, bmsfootprints:SOT95P237X102-3N, F.Cu at (167.9, 65.9)
- added Q11: SI2318DS-T1-E3, bmsfootprints:SOT95P237X102-3N, F.Cu at (172.8, 61.3)
- added Q12: SI2318DS-T1-E3, bmsfootprints:SOT95P237X102-3N, F.Cu at (172.8, 65.9)
- added Q2: SI2318DS-T1-E3, bmsfootprints:SI2318DS-T1-E3, F.Cu at (158.0, 65.9)
- added Q3: SI2318DS-T1-E3, bmsfootprints:SI2318DS-T1-E3, F.Cu at (162.9, 61.3)
- added Q4: SI2318DS-T1-E3, bmsfootprints:SI2318DS-T1-E3, F.Cu at (162.9, 65.9)
- added Q5: AONS66614, bmsfootprints:AON6482, F.Cu at (126.4, 63.6)
- added Q6: AONS66614, bmsfootprints:AON6482, F.Cu at (134.7, 63.6)
- added Q7: AONS66614, bmsfootprints:AON6482, F.Cu at (143.0, 63.6)
- added Q8: AONS66614, bmsfootprints:AON6482, F.Cu at (151.3, 63.6)
- added Q9: SI2318DS-T1-E3, bmsfootprints:SOT95P237X102-3N, F.Cu at (167.9, 61.3)
- added R11: 10, Resistor_SMD:R_0603_1608Metric, F.Cu at (158.1, 82.1)
- added R12: 10, Resistor_SMD:R_0603_1608Metric, F.Cu at (158.1, 84.6)
- added R14: 10, Resistor_SMD:R_0603_1608Metric, F.Cu at (162.1, 69.5)
- added R16: 10k, Resistor_SMD:R_0603_1608Metric, F.Cu at (162.1, 72.0)
- added R17: 10k, Resistor_SMD:R_0603_1608Metric, F.Cu at (162.1, 74.5)
- added R18: 10k, Resistor_SMD:R_0603_1608Metric, F.Cu at (162.1, 77.1)
- added R19: 10k, Resistor_SMD:R_0603_1608Metric, F.Cu at (162.1, 79.6)
- added R20: 10k, Resistor_SMD:R_0603_1608Metric, F.Cu at (162.1, 82.1)
- added R21: 10k, Resistor_SMD:R_0603_1608Metric, F.Cu at (162.1, 84.6)
- added R22: 10k, Resistor_SMD:R_0603_1608Metric, F.Cu at (166.1, 69.5)
- added R24: 30.1k, Resistor_SMD:R_0402_1005Metric, F.Cu at (136.4, 97.0)
- added R25: 5.23k, Resistor_SMD:R_0603_1608Metric, F.Cu at (166.1, 72.0)
- added R26: 10k, Resistor_SMD:R_0603_1608Metric, F.Cu at (166.1, 74.5)
- added R30: 10, Resistor_SMD:R_0603_1608Metric, F.Cu at (166.1, 77.1)
- added R4: 10, Resistor_SMD:R_0603_1608Metric, F.Cu at (158.1, 79.6)
- added RR_BATT_SNS1: 5m, Resistor_SMD:R_1206_3216Metric, F.Cu at (170.5, 87.5)
- added RT1: 103AT-2, bmsfootprints:103AT-2, F.Cu at (152.2, 93.8)
- added R_AC1: 1M, Resistor_SMD:R_0201_0603Metric, F.Cu at (166.5, 99.0)
- added R_AC2: 11.83k, Resistor_SMD:R_0603_1608Metric, F.Cu at (166.1, 79.6)
- added R_AC3: 53.25, Resistor_SMD:R_1206_3216Metric, F.Cu at (170.5, 90.8)
- added R_AC_SNS1: 5m, Resistor_SMD:R_1206_3216Metric, F.Cu at (170.5, 94.1)
- added R_FB1: 249k, Resistor_SMD:R_0402_1005Metric, F.Cu at (136.4, 99.0)
- added R_FBG1: 16.67k, Resistor_SMD:R_0603_1608Metric, F.Cu at (166.1, 82.1)
- added R_FSW_SYNC1: 40k, Resistor_SMD:R_0402_1005Metric, F.Cu at (136.4, 100.9)
- added R_ICHG1: 16.67k, Resistor_SMD:R_0603_1608Metric, F.Cu at (166.1, 84.6)
- added R_ILIM_HIZ1: 25k, Resistor_SMD:R_0402_1005Metric, F.Cu at (136.4, 102.9)
- added SW1: 100SP1T1B1M1QEH, bmsfootprints:SW_100SP1T1B1M1QEH, F.Cu at (129.4, 91.2)
- added U1: BQ25756ERRVR, bmsfootprints:IC_BQ25756ERRVR, F.Cu at (171.6, 99.8)
