File: hardware/Charge Controller Files (Michael:Sky)/ChargeController2.0.kicad_pcb (KiCad board)
At the start: 2 copper layers, 90.2 x 95.9 mm, 90 parts, among them J1 GND_TEST_01x01_Pin, J10 SOL_TEST_01x01_Pin, J13 Conn-1x2, J14 Conn-1x2, J15 Conn-1x2, J17 SCL_MAS_01x01_Pin, J18 SDA_MAS_01x01_Pin, J19 SYS-1x2, J2 SP_01x02_Pin, J3 BATT_TEST_01x01_Pin, J4 3.3V_PULLUP_01x02_Pin, J5 BATT_01x02_Pin, J6 Conn-1x2, J7 Conn-1x2, J8 Conn-1x2, J9 SYS_TEST_01x01_Pin, Q1 SI2318CDS-T1-GE3, Q10 SI2318CDS-T1-GE3, Q11 SI2318CDS-T1-GE3, Q12 SI2318CDS-T1-GE3, Q2 SI2318CDS-T1-GE3, Q3 SI2318CDS-T1-GE3, Q4 SI2318CDS-T1-GE3, Q5 AONS66614, Q6 AONS66614, Q7 AONS66614, Q8 AONS66614, Q9 SI2318CDS-T1-GE3, SW1 100SP1T1B1M1QEH, U1 BQ25756ERRVR

Commit message: Charge Controller 3.0
Next Prototype formatting (Schematic Format Done)
Parts:
- removed C12, C13, C17, C18, C2, C24: 56u, Capacitor_SMD:C_0201_0603Metric
- removed C14, C16, C19, C20, C25, C27, C4: 100n, Capacitor_SMD:C_0402_1005Metric
- removed C15, C26: 470n, Capacitor_SMD:C_0402_1005Metric
- removed C22, C3, C7: 4.7u, Capacitor_SMD:C_0603_1608Metric
- removed C23: 1u, Capacitor_SMD:C_0201_0603Metric
- removed C6: 47u, Capacitor_SMD:C_0603_1608Metric
- removed D1, D2, D3: GREEN, LED_SMD:LED_0603_1608Metric
- removed D4, D5: BAT54, bmsfootprints:BAT54
- removed D6, D7, D8, D9: SS24, bmsfootprints:SS24
- removed H1, H2, H3, H4: MountingHole_Pad, MountingHole:MountingHole_3.2mm_M3_ISO14580_Pad
- removed J1: GND_TEST_01x01_Pin, Connector_PinHeader_2.54mm:PinHeader_1x01_P2.54mm_Vertical
- removed J10: SOL_TEST_01x01_Pin, Connector_PinHeader_2.54mm:PinHeader_1x01_P2.54mm_Vertical
- removed J13, J14, J15, J6, J7, J8: Conn-1x2, Connector_PinHeader_2.54mm:PinHeader_1x02_P2.54mm_Vertical
- removed J17: SCL_MAS_01x01_Pin, Connector_PinHeader_2.54mm:PinHeader_1x01_P2.54mm_Vertical
- removed J18: SDA_MAS_01x01_Pin, Connector_PinHeader_2.54mm:PinHeader_1x01_P2.54mm_Vertical
- removed J19: SYS-1x2, Connector_PinHeader_2.54mm:PinHeader_1x02_P2.54mm_Vertical
- removed J2: SP_01x02_Pin, Connector_PinHeader_2.54mm:PinHeader_1x02_P2.54mm_Vertical
- removed J3: BATT_TEST_01x01_Pin, Connector_PinHeader_2.54mm:PinHeader_1x01_P2.54mm_Vertical
- removed J4: 3.3V_PULLUP_01x02_Pin, Connector_PinHeader_2.54mm:PinHeader_1x02_P2.54mm_Vertical
- removed J5: BATT_01x02_Pin, Connector_PinHeader_2.54mm:PinHeader_1x02_P2.54mm_Vertical
- removed J9: SYS_TEST_01x01_Pin, Connector_PinHeader_2.54mm:PinHeader_1x01_P2.54mm_Vertical
- removed L1: IHLP6767GZER100M01, bmsfootprints:IND_IHLP6767GZER100M01
- removed Q1, Q10, Q11, Q12, Q2, Q3, Q4, Q9: SI2318CDS-T1-GE3, bmsfootprints:SI2318CDS-T1-GE3
- removed Q5, Q6, Q7, Q8: AONS66614, bmsfootprints:AON6482
- removed R11, R12, R14, R30, R4: 10, Resistor_SMD:R_0603_1608Metric
- removed R16, R17, R18, R19, R20, R21, R22, R26: 10k, Resistor_SMD:R_0603_1608Metric
- removed R24: 30.1k, Resistor_SMD:R_0402_1005Metric
- removed R25: 5.23k, Resistor_SMD:R_0603_1608Metric
- removed RR_BATT_SNS1, R_AC_SNS1: 5m, Resistor_SMD:R_1206_3216Metric
- removed RT1: 103AT-2, bmsfootprints:103AT-2
- removed R_AC1: 1M, Resistor_SMD:R_0201_0603Metric
- removed R_AC2: 11.83k, Resistor_SMD:R_0603_1608Metric
- removed R_AC3: RC0402FR-0753K6L, bmsfootprints:RC0402FR-0753K6L
- removed R_FB1: 249k, Resistor_SMD:R_0402_1005Metric
- removed R_FBG1, R_ICHG1: 16.67k, Resistor_SMD:R_0603_1608Metric
- removed R_FSW_SYNC1: 40k, Resistor_SMD:R_0402_1005Metric
- removed R_ILIM_HIZ1: 25k, Resistor_SMD:R_0402_1005Metric
- removed SW1: 100SP1T1B1M1QEH, bmsfootprints:SW_100SP1T1B1M1QEH
- removed U1: BQ25756ERRVR, bmsfootprints:IC_BQ25756ERRVR
Routing:
- net /EN: track 126.0 -> 0.00 mm, vias 9 -> 0
- net Net-(C17-Pad1): track 115.9 -> 0.00 mm, vias 2 -> 0
- net GND: track 80.5 -> 0.00 mm, vias 37 -> 0
- net VAC: track 55.3 -> 0.00 mm
- net /TS: track 53.9 -> 0.00 mm
- net PGND: track 52.0 -> 0.00 mm, vias 2 -> 0
- net Net-(J4-Pin_1): track 51.2 -> 0.00 mm
- net Net-(D6-PadC): track 50.8 -> 0.00 mm
- net /DRV_SUP: track 49.1 -> 0.00 mm, vias 4 -> 0
- net /SW1: track 43.2 -> 0.00 mm, vias 2 -> 0
- net /SW2: track 36.5 -> 0.00 mm, vias 2 -> 0
- net Net-(Q6-D_1): track 32.3 -> 0.00 mm, vias 2 -> 0
- net /CE: track 30.4 -> 0.00 mm
- net /PG: track 29.5 -> 0.00 mm
- net /HIDRV_1: track 28.6 -> 0.00 mm
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- removed copper zone on B.Cu, net GND
Other:
- board outline removed
- board text removed: "Charge Controller 2.0 - Michael Petta, Sky Lin"
- board text removed: "Husky Satellite Lab"

Commit message: Fix?
Fix?
Parts:
- added C12: 56u, Capacitor_SMD:C_0201_0603Metric, F.Cu at (157.0, 91.7)
- added C13: 56u, Capacitor_SMD:C_0201_0603Metric, F.Cu at (149.5, 103.3)
- added C14: 100n, Capacitor_SMD:C_0402_1005Metric, F.Cu at (193.0, 96.5)
- added C15: 470n, Capacitor_SMD:C_0402_1005Metric, F.Cu at (190.5, 97.0)
- added C16: 100n, Capacitor_SMD:C_0402_1005Metric, F.Cu at (188.0, 96.5)
- added C17: 56u, Capacitor_SMD:C_0201_0603Metric, F.Cu at (199.0, 107.5)
- added C18: 56u, Capacitor_SMD:C_0201_0603Metric, F.Cu at (196.0, 107.5)
- added C19: 100n, Capacitor_SMD:C_0402_1005Metric, F.Cu at (172.0, 93.0)
- added C2: 56u, Capacitor_SMD:C_0201_0603Metric, F.Cu at (152.5, 105.5)
- added C20: 100n, Capacitor_SMD:C_0402_1005Metric, F.Cu at (189.0, 93.0)
- added C22: 4.7u, Capacitor_SMD:C_0603_1608Metric, F.Cu at (184.8, 88.0)
- added C23: 1u, Capacitor_SMD:C_0201_0603Metric, F.Cu at (165.5, 105.0)
- added C24: 56u, Capacitor_SMD:C_0201_0603Metric, F.Cu at (195.3, 98.0)
- added C25: 100n, Capacitor_SMD:C_0402_1005Metric, F.Cu at (177.5, 95.0)
- added C26: 470n, Capacitor_SMD:C_0402_1005Metric, F.Cu at (172.0, 96.0)
- added C27: 100n, Capacitor_SMD:C_0402_1005Metric, F.Cu at (164.2, 97.1)
- added C3: 4.7u, Capacitor_SMD:C_0603_1608Metric, F.Cu at (182.5, 90.5)
- added C4: 100n, Capacitor_SMD:C_0402_1005Metric, F.Cu at (162.5, 105.0)
- added C6: 47u, Capacitor_SMD:C_0603_1608Metric, F.Cu at (158.0, 109.0)
- added C7: 4.7u, Capacitor_SMD:C_0603_1608Metric, F.Cu at (156.0, 105.7)
- added D1: GREEN, LED_SMD:LED_0603_1608Metric, F.Cu at (193.5, 125.3)
- added D2: GREEN, LED_SMD:LED_0603_1608Metric, F.Cu at (184.5, 123.8)
- added D3: GREEN, LED_SMD:LED_0603_1608Metric, F.Cu at (189.0, 123.8)
- added D4: BAT54, bmsfootprints:BAT54, F.Cu at (196.5, 94.0)
- added D5: BAT54, bmsfootprints:BAT54, F.Cu at (165.1, 93.0)
- added D6: SS24, bmsfootprints:SS24, F.Cu at (143.0, 106.8)
- added D7: SS24, bmsfootprints:SS24, F.Cu at (143.0, 51.7)
- added D8: SS24, bmsfootprints:SS24, F.Cu at (162.8, 42.5)
- added D9: SS24, bmsfootprints:SS24, F.Cu at (162.8, 50.0)
- added H1: MountingHole_Pad, MountingHole:MountingHole_3.2mm_M3_ISO14580_Pad, F.Cu at (222.1, 41.6)
- added H2: MountingHole_Pad, MountingHole:MountingHole_3.2mm_M3_ISO14580_Pad, F.Cu at (222.1, 127.3)
- added H3: MountingHole_Pad, MountingHole:MountingHole_3.2mm_M3_ISO14580_Pad, F.Cu at (142.1, 127.3)
- added H4: MountingHole_Pad, MountingHole:MountingHole_3.2mm_M3_ISO14580_Pad, F.Cu at (142.1, 41.6)
- added J1: GND_TEST_01x01_Pin, Connector_PinHeader_2.54mm:PinHeader_1x01_P2.54mm_Vertical, F.Cu at (148.5, 127.0)
- added J10: SOL_TEST_01x01_Pin, Connector_PinHeader_2.54mm:PinHeader_1x01_P2.54mm_Vertical, F.Cu at (148.5, 117.5)
- added J13: Conn-1x2, Connector_PinHeader_2.54mm:PinHeader_1x02_P2.54mm_Vertical, F.Cu at (197.0, 120.5)
- added J14: Conn-1x2, Connector_PinHeader_2.54mm:PinHeader_1x02_P2.54mm_Vertical, F.Cu at (180.0, 116.5)
- added J15: Conn-1x2, Connector_PinHeader_2.54mm:PinHeader_1x02_P2.54mm_Vertical, F.Cu at (184.0, 116.5)
- added J17: SCL_MAS_01x01_Pin, Connector_PinHeader_2.54mm:PinHeader_1x01_P2.54mm_Vertical, F.Cu at (172.0, 118.0)
- added J18: SDA_MAS_01x01_Pin, Connector_PinHeader_2.54mm:PinHeader_1x01_P2.54mm_Vertical, F.Cu at (176.0, 118.0)
- added J19: SYS-1x2, Connector_PinHeader_2.54mm:PinHeader_1x02_P2.54mm_Vertical, F.Cu at (204.0, 40.0)
- added J2: SP_01x02_Pin, Connector_PinHeader_2.54mm:PinHeader_1x02_P2.54mm_Vertical, F.Cu at (143.0, 115.0)
- added J3: BATT_TEST_01x01_Pin, Connector_PinHeader_2.54mm:PinHeader_1x01_P2.54mm_Vertical, F.Cu at (180.5, 41.0)
- added J4: 3.3V_PULLUP_01x02_Pin, Connector_PinHeader_2.54mm:PinHeader_1x02_P2.54mm_Vertical, F.Cu at (206.8, 128.0)
- added J5: BATT_01x02_Pin, Connector_PinHeader_2.54mm:PinHeader_1x02_P2.54mm_Vertical, F.Cu at (173.5, 40.2)
- added J6: Conn-1x2, Connector_PinHeader_2.54mm:PinHeader_1x02_P2.54mm_Vertical, F.Cu at (211.7, 98.5)
- added J7: Conn-1x2, Connector_PinHeader_2.54mm:PinHeader_1x02_P2.54mm_Vertical, F.Cu at (202.0, 95.7)
- added J8: Conn-1x2, Connector_PinHeader_2.54mm:PinHeader_1x02_P2.54mm_Vertical, F.Cu at (216.0, 109.0)
- added J9: SYS_TEST_01x01_Pin, Connector_PinHeader_2.54mm:PinHeader_1x01_P2.54mm_Vertical, F.Cu at (210.5, 40.0)
- added L1: IHLP6767GZER100M01, bmsfootprints:IND_IHLP6767GZER100M01, F.Cu at (181.5, 74.0)
- added Q1: SI2318CDS-T1-GE3, bmsfootprints:SI2318CDS-T1-GE3, F.Cu at (143.0, 98.5)
- added Q10: SI2318CDS-T1-GE3, bmsfootprints:SI2318CDS-T1-GE3, F.Cu at (196.5, 41.0)
- added Q11: SI2318CDS-T1-GE3, bmsfootprints:SI2318CDS-T1-GE3, F.Cu at (188.5, 41.0)
- added Q12: SI2318CDS-T1-GE3, bmsfootprints:SI2318CDS-T1-GE3, F.Cu at (150.4, 92.0)
- added Q2: SI2318CDS-T1-GE3, bmsfootprints:SI2318CDS-T1-GE3, F.Cu at (143.0, 91.5)
- added Q3: SI2318CDS-T1-GE3, bmsfootprints:SI2318CDS-T1-GE3, F.Cu at (174.1, 50.0)
- added Q4: SI2318CDS-T1-GE3, bmsfootprints:SI2318CDS-T1-GE3, F.Cu at (182.0, 49.5)
- added Q5: AONS66614, bmsfootprints:AON6482, F.Cu at (159.0, 86.0)
- added Q6: AONS66614, bmsfootprints:AON6482, F.Cu at (205.2, 86.4)
- added Q7: AONS66614, bmsfootprints:AON6482, F.Cu at (167.4, 81.7)
- added Q8: AONS66614, bmsfootprints:AON6482, F.Cu at (195.7, 83.4)
- added Q9: SI2318CDS-T1-GE3, bmsfootprints:SI2318CDS-T1-GE3, F.Cu at (191.1, 49.5)
- added R11: 10, Resistor_SMD:R_0603_1608Metric, F.Cu at (175.5, 97.2)
- added R12: 10, Resistor_SMD:R_0603_1608Metric, F.Cu at (192.0, 99.5)
- added R14: 10, Resistor_SMD:R_0603_1608Metric, F.Cu at (188.5, 99.5)
- added R16: 10k, Resistor_SMD:R_0603_1608Metric, F.Cu at (172.2, 124.0)
- added R17: 10k, Resistor_SMD:R_0603_1608Metric, F.Cu at (176.2, 124.0)
- added R18: 10k, Resistor_SMD:R_0603_1608Metric, F.Cu at (201.5, 121.5)
- added R19: 10k, Resistor_SMD:R_0603_1608Metric, F.Cu at (198.0, 126.5)
- added R20: 10k, Resistor_SMD:R_0603_1608Metric, F.Cu at (180.2, 123.5)
- added R21: 10k, Resistor_SMD:R_0603_1608Metric, F.Cu at (184.7, 128.5)
- added R22: 10k, Resistor_SMD:R_0603_1608Metric, F.Cu at (189.0, 128.5)
- added R24: 30.1k, Resistor_SMD:R_0402_1005Metric, F.Cu at (220.5, 107.0)
- added R25: 5.23k, Resistor_SMD:R_0603_1608Metric, F.Cu at (207.0, 100.0)
- added R26: 10k, Resistor_SMD:R_0603_1608Metric, F.Cu at (220.5, 103.7)
- added R30: 10, Resistor_SMD:R_0603_1608Metric, F.Cu at (168.5, 96.5)
- added R4: 10, Resistor_SMD:R_0603_1608Metric, F.Cu at (159.5, 105.7)
- added RR_BATT_SNS1: 5m, Resistor_SMD:R_1206_3216Metric, F.Cu at (194.5, 103.5)
- added RT1: 103AT-2, bmsfootprints:103AT-2, F.Cu at (216.0, 103.5)
- added R_AC1: 1M, Resistor_SMD:R_0201_0603Metric, F.Cu at (169.5, 102.0)
- added R_AC2: 11.83k, Resistor_SMD:R_0603_1608Metric, F.Cu at (170.5, 105.5)
- added R_AC3: RC0402FR-0753K6L, bmsfootprints:RC0402FR-0753K6L, F.Cu at (175.0, 105.0)
- added R_AC_SNS1: 5m, Resistor_SMD:R_1206_3216Metric, F.Cu at (172.5, 100.0)
- added R_FB1: 249k, Resistor_SMD:R_0402_1005Metric, F.Cu at (190.5, 102.5)
- added R_FBG1: 16.67k, Resistor_SMD:R_0603_1608Metric, F.Cu at (187.7, 103.5)
- added R_FSW_SYNC1: 40k, Resistor_SMD:R_0402_1005Metric, F.Cu at (174.0, 110.5)
- added R_ICHG1: 16.67k, Resistor_SMD:R_0603_1608Metric, F.Cu at (192.5, 109.0)
- added R_ILIM_HIZ1: 25k, Resistor_SMD:R_0402_1005Metric, F.Cu at (189.5, 106.5)
- added SW1: 100SP1T1B1M1QEH, bmsfootprints:SW_100SP1T1B1M1QEH, F.Cu at (152.5, 46.0)
- added U1: BQ25756ERRVR, bmsfootprints:IC_BQ25756ERRVR, F.Cu at (182.5, 97.0)
Routing:
- net /EN: track 0.00 -> 126.0 mm, vias 0 -> 9
- net Net-(C17-Pad1): track 0.00 -> 115.9 mm, vias 0 -> 2
- net GND: track 0.00 -> 80.5 mm, vias 0 -> 37
- net VAC: track 0.00 -> 55.3 mm
- net /TS: track 0.00 -> 53.9 mm
- net PGND: track 0.00 -> 52.0 mm, vias 0 -> 2
- net Net-(J4-Pin_1): track 0.00 -> 51.2 mm
- net Net-(D6-PadC): track 0.00 -> 50.8 mm
- net /DRV_SUP: track 0.00 -> 49.1 mm, vias 0 -> 4
- net /SW1: track 0.00 -> 43.2 mm, vias 0 -> 2
- net /SW2: track 0.00 -> 36.5 mm, vias 0 -> 2
- net Net-(Q6-D_1): track 0.00 -> 32.3 mm, vias 0 -> 2
- net /CE: track 0.00 -> 30.4 mm
- net /PG: track 0.00 -> 29.5 mm
- net /HIDRV_1: track 0.00 -> 28.6 mm
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- added copper zone on B.Cu, net GND
Other:
- board outline added: 90.2 x 95.9 mm
- board text added: "Charge Controller 2.0 - Michael Petta, Sky Lin"
- board text added: "Husky Satellite Lab"
