File: hardware/Charge Controller 3.0 Files (Michael_Sky)/ChargeController3.0/TempManager.kicad_sch (KiCad schematic)
At the start: 7 parts, among them J6 Conn-1x2, J7 Conn-1x2, J8 Conn-1x2

Commit message: New formatting
New formatting
Parts:
- removed J6, J7, J8: Conn-1x2, Connector_PinHeader_2.54mm:PinHeader_1x02_P2.54mm_Vertical, symbol Connector:Conn_01x02_Pin
- removed R26: 10k, Resistor_SMD:R_0603_1608Metric, symbol Device:R
Connections:
- net GND: now also RT1.2
- net REGN: now also R25.2
Other:
- moved on the sheet: RT1
