File: hardware/Charge Controller 3.0 Files (Michael_Sky)/ChargeController3.0/ChargeController3.0.kicad_pcb (KiCad board)
At the start: 2 copper layers, 95.9 x 90.2 mm, 96 parts, among them J1 Conn_02x26_Odd_Even, J12 Conn_02x26_Odd_Even, J20 Conn_01x08_Pin, J4 3.3V_PULLUP_01x02_Pin, Q12 SOT91P240X110-3N, Q13 SOT91P240X110-3N, Q5 AONS66614, Q6 AONS66614, Q7 AONS66614, Q8 AONS66614, SW1 100SP1T1B1M1QEH, U1 BQ25756ERRVR, U10 BAT46WJ_115, U11 BAT46WJ_115, U2 SISH101DN-T1-GE3, U3 SISH101DN-T1-GE3, U4 SISH101DN-T1-GE3, U5 SI4122DY-T1-GE3, U6 SI4122DY-T1-GE3, U7 SISH101DN-T1-GE3, U8 SISH101DN-T1-GE3, U9 BAT46WJ_115

Commit message: librecube edits
edits
Parts:
- moved H2 3.81 mm to (194.8, 68.8)
Routing:
- net Net-(C9-Pad1): track 11.6 -> 15.8 mm
Changed lines of the file:
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@@
 	(footprint "MountingHole:MountingHole_3.2mm_M3_ISO14580_Pad"
 		(layer "F.Cu")
-		(at 194.81 65.03)
+		(at 194.81 68.84)
 		(descr "Mounting Hole 3.2mm, M3, generated by kicad-footprint-generator mountinghole.py")
 		(tags "mountinghole M3 ISO14580")
@@
 	)
 	(segment
-		(start 194.81 65.03)
-		(end 192.78 63)
+		(start 192.37 66.4)
+		(end 189.64 66.4)
 		(width 0.2)
 		(layer "F.Cu")
@@
 	)
 	(segment
-		(start 193.44 66.4)
-		(end 194.81 65.03)
+		(start 192.78 66.81)
+		(end 194.81 68.84)
 		(width 0.2)
 		(layer "F.Cu")
@@
 	)
 	(segment
-		(start 189.64 66.4)
-		(end 193.44 66.4)
+		(start 194.81 68.84)
+		(end 192.37 66.4)
 		(width 0.2)
 		(layer "F.Cu")
@@
 	)
 	(segment
+		(start 192.78 63)
+		(end 192.78 66.81)
+		(width 0.2)
+		(layer "F.Cu")
+		(net "Net-(C9-Pad1)")
+	)
+	(segment
 		(start 159.12 107.6)
 		(end 159.12 107.1)
@@
 		(polygon
 			(pts
-				(xy 103.45 59.7) (xy 199.8 59.55) (xy 199.95 150.3) (xy 103.95 150.15) (xy 103.45 59.65)
+				(xy 103.7 60.8) (xy 105.3 59.2) (xy 141.5 59.3) (xy 143 61.7) (xy 161.2 61.7) (xy 162.1 60.1) (xy 198.8 59.8)
+				(xy 200.1 61.1) (xy 200.1 95) (xy 199.1 96.1) (xy 197.7 96.1) (xy 197.3 99) (xy 197.3 115.4) (xy 198.6 116.2)
+				(xy 199.8 116.3) (xy 200.1 148.7) (xy 198.6 150.5) (xy 103.9 151) (xy 104 116.1) (xy 106.4 116)
+				(xy 106.8 96.5) (xy 103.5 94.6) (xy 103.4 60.6)
 			)
 		)
